File: hardware/mcu.kicad_sch (KiCad schematic)
At the start: 0 parts

Commit message: Split the TMC2209 wiring by bare IC vs module
The driver table assumed a SilentStepStick, which hides the charge pump, sense
resistors and regulator capacitors on the module. A bare QFN-28 needs all of
them externally, and the pins involved are not optional: VS, VCP, CPI/CPO and
5VOUT drive the charge pump that generates high-side gate drive, and BRA/BRB
are the current sense returns.

Documents both cases, with the pin names that tell them apart, and notes the
real cost of bare ICs - about eight passives per driver, forty across the
board. Only DIAG, INDEX and NC are genuinely No-Connect either way.
Parts:
- added U1: ESP32-S3-WROOM-1, RF_Module:ESP32-S3-WROOM-1, symbol RF_Module:ESP32-S3-WROOM-1
Connections:
- new net +3V3: U1.2 (3V3)
- new net GND: U1.1 (GND), U1.40 (GND), U1.41 (GND)
- no-connect marks 0 -> 3
