File: hardware/usb.kicad_sch (KiCad schematic)
At the start: 3 parts, among them P1 USB_C_Plug_USB2.0

Commit message: Add JLCPCB assembly path for the buck
The Recom module is SIP-3 through-hole and unlikely to be in JLC's library.
Documents two routes: mark it DNP and hand-solder three pins after assembly,
which keeps the 72 V margin and one-part simplicity; or switch to an SMD part
JLC stocks.

Lists selection criteria and three candidates to check against the live parts
library - LM2675MX-5.0 (best if stocked), XL1509-5.0E1 (cheap, near-certain
LCSC stock, but 150 kHz means a bulky inductor), and MP4560 (55 V, better
margin). Notes that stock cannot be verified from here.
Parts:
- D1: value D_Schottky -> SS34; footprint (none) -> Diode_SMD:D_SMA
Connections:
- net at P1.A4 (VBUS), P1.A9 (VBUS), P1.B4 (VBUS)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: now also D1.2 (A); no longer D1.1 (K)
- new net +5V: D1.1 (K)
Other:
- moved on the sheet: D1
Changed lines of the file:
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@@
+	(wire
+		(pts
+			(xy 149.86 59.69) (xy 138.43 59.69)
+		)
+		(stroke
+			(width 0)
+			(type default)
+		)
+	)
 	(wire
 		(pts
@@
 	)
 	(symbol
+		(lib_id "power:+5V")
+		(at 149.86 59.69 0)
+		(unit 1)
+		(body_style 1)
+		(exclude_from_sim no)
+		(in_bom yes)
+		(on_board yes)
+		(in_pos_files yes)
+		(dnp no)
+		(fields_autoplaced yes)
+		(property "Reference" "#PWR035"
+			(at 149.86 63.5 0)
+			(hide yes)
+			(show_name no)
+			(do_not_autoplace no)
+			(effects
+				(font
+					(size 1.27 1.27)
+				)
+			)
+		)
+		(property "Value" "+5V"
+			(at 149.86 54.61 0)
+			(show_name no)
+			(do_not_autoplace no)
+			(effects
+				(font
+					(size 1.27 1.27)
+				)
+			)
+		)
+		(property "Footprint" ""
+			(at 149.86 59.69 0)
+			(hide yes)
+			(show_name no)
+			(do_not_autoplace no)
+			(effects
+				(font
+					(size 1.27 1.27)
+				)
+			)
+		)
+		(property "Datasheet" ""
+			(at 149.86 59.69 0)
+			(hide yes)
+			(show_name no)
+			(do_not_autoplace no)
+			(effects
+				(font
+					(size 1.27 1.27)
+				)
+			)
+		)
+		(property "Description" "Power symbol creates a global label with name \"+5V\""
+			(at 149.86 59.69 0)
+			(hide yes)
+			(show_name no)
+			(do_not_autoplace no)
+			(effects
+				(font
+					(size 1.27 1.27)
+				)
+			)
+		)
+		(pin "1"
+		)
+		(instances
+			(project "ufluidics"
+				(path "/bf8ba2d7-3b7b-4865-bab6-5f38b618ecb0/2d60a5db-c1d2-4142-924d-8a10382c57fd"
+					(reference "#PWR035")
+					(unit 1)
+				)
+			)
+		)
+	)
+	(symbol
 		(lib_id "power:GND")
 		(at 147.32 67.31 0)
@@
 	(symbol
 		(lib_id "Device:D_Schottky")
-		(at 134.62 59.69 0)
+		(at 134.62 59.69 180)
 		(unit 1)
 		(body_style 1)
@@
 		(fields_autoplaced yes)
 		(property "Reference" "D1"
-			(at 134.3025 53.34 0)
-			(show_name no)
-			(do_not_autoplace no)
-			(effects
-				(font
-					(size 1.27 1.27)
-				)
-			)
-		)
-		(property "Value" "D_Schottky"
-			(at 134.3025 55.88 0)
-			(show_name no)
-			(do_not_autoplace no)
-			(effects
-				(font
-					(size 1.27 1.27)
-				)
-			)
-		)
-		(property "Footprint" ""
+			(at 134.9375 53.34 0)
+			(show_name no)
+			(do_not_autoplace no)
+			(effects
+				(font
+					(size 1.27 1.27)
+				)
+			)
+		)
+		(property "Value" "SS34"
+			(at 134.9375 55.88 0)
+			(show_name no)
+			(do_not_autoplace no)
+			(effects
+				(font
+					(size 1.27 1.27)
+				)
+			)
+		)
+		(property "Footprint" "Diode_SMD:D_SMA"
 			(at 134.62 59.69 0)
 			(hide yes)
