File: hardware/ufluidics.kicad_sch (KiCad schematic)
At the start: 17 parts, among them J19 Conn_01x04, J20 Conn_01x09, U1 ESP32-S3-WROOM-1

Commit message: route
Parts:
- added J21: Conn_01x02, Connector_PinHeader_2.54mm:PinHeader_1x02_P2.54mm_Vertical, symbol Connector_Generic:Conn_01x02
Connections:
- net LED_RUN: now also U1.15 (IO3); no longer U1.26 (IO45)
- net POT_A: now also U1.38 (IO2); no longer U1.39 (IO1)
- net POT_B: now also U1.39 (IO1); no longer U1.38 (IO2)
- net GPIO14: now reaches U1.22 (IO14)
- net GPIO14: now also J21.1 (Pin_1)
- new net GPIO45: J21.2 (Pin_2), U1.26 (IO45)
- no-connect marks 3 -> 1
Other:
- note added: "Extra Pins"
Changed lines of the file:
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@@
 	)
 	(rectangle
+		(start 25.4 178.435)
+		(end 71.12 194.945)
+		(stroke
+			(width 0)
+			(type default)
+		)
+		(fill
+			(type none)
+		)
+	)
+	(rectangle
 		(start 25.4 17.78)
 		(end 71.12 52.705)
@@
 		)
 	)
+	(text "Extra Pins"
+		(exclude_from_sim no)
+		(at 26.416 193.294 0)
+		(effects
+			(font
+				(size 1.27 1.27)
+			)
+			(justify left)
+		)
+	)
 	(text "Switch, enables and disables stepper drivers. \nDoes not cut power to MCU"
 		(exclude_from_sim no)
@@
 	)
 	(no_connect
-		(at 93.98 72.39)
-	)
-	(no_connect
-		(at 93.98 44.45)
-	)
-	(no_connect
 		(at 222.25 52.07)
 	)
@@
 		)
 	)
-	(label "USB_D_P"
-		(at 265.43 52.07 0)
+	(label "LED_RUN"
+		(at 93.98 44.45 180)
 		(effects
 			(font
 				(size 1.27 1.27)
 			)
-			(justify left bottom)
+			(justify right bottom)
 		)
 	)
-	(label "LED_RUN"
-		(at 124.46 69.85 0)
+	(label "GPIO14"
+		(at 46.99 185.42 180)
+		(effects
+			(font
+				(size 1.27 1.27)
+			)
+			(justify right bottom)
+		)
+	)
+	(label "USB_D_P"
+		(at 265.43 52.07 0)
 		(effects
 			(font
@@
 		)
 	)
+	(label "GPIO14"
+		(at 93.98 72.39 180)
+		(effects
+			(font
+				(size 1.27 1.27)
+			)
+			(justify right bottom)
+		)
+	)
 	(label "BOOT"
 		(at 93.98 36.83 180)
@@
 		)
 	)
-	(label "POT_A"
-		(at 93.98 39.37 180)
+	(label "GPIO45"
+		(at 46.99 187.96 180)
 		(effects
 			(font
@@
 		)
 	)
+	(label "GPIO45"
+		(at 124.46 69.85 0)
+		(effects
+			(font
+				(size 1.27 1.27)
+			)
+			(justify left bottom)
+		)
+	)
 	(label "USB_D_P"
 		(at 124.46 44.45 0)
@@
 		)
 	)
-	(label "TMC_UART_A"
-		(at 166.37 85.09 180)
+	(label "POT_B"
+		(at 93.98 39.37 180)
 		(effects
 			(font
@@
 		)
 	)
-	(label "I2C_SDA"
-		(at 220.98 111.76 180)
+	(label "TMC_UART_A"
+		(at 166.37 85.09 180)
 		(effects
 			(font
@@
 		)
 	)
-	(label "POT_B"
-		(at 93.98 41.91 180)
+	(label "I2C_SDA"
+		(at 220.98 111.76 180)
 		(effects
 			(font
@@
 		)
 	)
+	(label "POT_A"
+		(at 93.98 41.91 180)
+		(effects
+			(font
+				(size 1.27 1.27)
+			)
+			(justify right bottom)
+		)
+	)
 	(label "IN2_DIR"
 		(at 93.98 49.53 180)
@@
 					(unit 1)
 				)
+			)
+		)
+	)
+	(symbol
+		(lib_id "Connector_Generic:Conn_01x02")
+		(at 52.07 185.42 0)
+		(unit 1)
+		(body_style 1)
+		(exclude_from_sim no)
+		(in_bom yes)
+		(on_board yes)
+		(in_pos_files yes)
+		(dnp no)
+		(fields_autoplaced yes)
+		(property "Reference" "J21"
+			(at 54.61 185.4199 0)
+			(show_name no)
+			(do_not_autoplace no)
+			(effects
+				(font
+					(size 1.27 1.27)
+				)
+				(justify left)
+			)
+		)
+		(property "Value" "Conn_01x02"
+			(at 54.61 187.9599 0)
+			(show_name no)
+			(do_not_autoplace no)
+			(effects
+				(font
+					(size 1.27 1.27)
+				)
+				(justify left)
+			)
+		)
+		(property "Footprint" "Connector_PinHeader_2.54mm:PinHeader_1x02_P2.54mm_Vertical"
+			(at 52.07 185.42 0)
+			(hide yes)
+			(show_name no)
+			(do_not_autoplace no)
+			(effects
+				(font
+					(size 1.27 1.27)
+				)
+			)
+		)
+		(property "Datasheet" ""
+			(at 52.07 185.42 0)
+			(hide yes)
+			(show_name no)
+			(do_not_autoplace no)
+			(effects
+				(font
+					(size 1.27 1.27)
+				)
+			)
+		)
+		(property "Description" "Generic connector, single row, 01x02, script generated (kicad-library-utils/schlib/autogen/connector/)"
+			(at 52.07 185.42 0)
+			(hide yes)
+			(show_name no)
+			(do_not_autoplace no)
+			(effects
+				(font
+					(size 1.27 1.27)
+				)
+			)
+		)
+		(pin "1"
+		)
+		(pin "2"
+		)
+		(instances
+			(project "ufluidics"
+				(path "/bf8ba2d7-3b7b-4865-bab6-5f38b618ecb0"
+					(reference "J21")
+					(unit 1)
+				)
